File: CampKeen_Galvanic_Tank_Sensor/CampKeen_Galvanic_Tank_Sensor.kicad_pcb (KiCad board)
At the start: 2 copper layers, 72.9 x 71.1 mm, 50 parts, among them IC2 OPA4340UA, J1 Power_And_CAN, J2 TankInputs, J3 TTL_Programmer, J4 ICSP, J5 Conn_02x02_Counter_Clockwise, J6 Screw_Terminal_01x02, Q1 IRF9Z34NPBF, Q30 2N7000, Q32 IRF9Z34NPBF, U1 3568, U2 ATmega328P-P, U3 MCP2515-xSO, U4 MCP2551-I-SN, U5 3568, Y1 16MHz, Y2 16MHz

Commit message: hardware looks to be done. routed and DRC'ed needs to be sent off to be fabbed.
Connections:
- J6 pad 2: Net-(J6-Pin_2) -> Net-(J6-Pin_1)
- U1 pad 1: Net-(J6-Pin_2) -> Net-(J6-Pin_1)
Routing:
- net +5V: track 0.00 -> 199.3 mm, vias 0 -> 1
- net GND: track 46.3 -> 214.0 mm, vias 3 -> 8
- net /BareMinAtmel328P/RESET: track 0.00 -> 105.5 mm, vias 0 -> 1
- net /BareMinAtmel328P/PB1-D9: track 0.00 -> 97.9 mm, vias 0 -> 3
- net Net-(U3-OSC1): track 0.00 -> 89.3 mm, vias 0 -> 3
- net Net-(U3-OSC2): track 0.00 -> 88.0 mm, vias 0 -> 4
- net /BareMinAtmel328P/PB4-D12-MISO: track 0.00 -> 81.9 mm, vias 0 -> 5
- net /BareMinAtmel328P/PC3-A3: track 0.00 -> 79.0 mm, vias 0 -> 5
- net /BareMinAtmel328P/PB3-D11-MOSI: track 0.00 -> 76.8 mm, vias 0 -> 4
- net /BareMinAtmel328P/PC0-A0: track 0.00 -> 69.8 mm, vias 0 -> 4
- net /BareMinAtmel328P/PC2-A2: track 0.00 -> 57.6 mm, vias 0 -> 1
- net /BareMinAtmel328P/PD1-TX: track 0.00 -> 55.9 mm, vias 0 -> 3
- net /BufferedADC/ADCIN4: track 0.00 -> 55.1 mm, vias 0 -> 4
- net /BareMinAtmel328P/PC1-A1: track 0.00 -> 54.3 mm, vias 0 -> 2
- net /BufferedADC/ADCIN1: track 0.00 -> 54.1 mm, vias 0 -> 4
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